File: hardware/PicoROM-28/PicoROM-28.kicad_sch (KiCad schematic)
At the start: 62 parts, among them J1 USB_C_Receptacle_USB2.0, J2 External Reset, J3 Conn_01x14, J4 Conn_01x14, J5 Conn_01x05_Pin, U1 NCP114AMX330TCG, U10 74LVC8245, U11 74AHCT1G126, U2 W25Q16JVUXIQ, U3 RP2040, U4 74LVC245, U5 74LVC245, U7 74AHCT1G126, U8 NCP114AMX330TCG, U9 74LVC245, Y1 ABM3-12.000MHZ-D2Y-T

Commit message: PicoROM-28 1.10-S: side-entry USB-C connector
Replace the vertical GT-USB-7051A USB-C receptacle (J1) with a horizontal
16-pin HRO TYPE-C-31-M-12 (LCSC C165948), so the plug enters from the
pin-1 end of the board instead of from above. Based on upstream 1.10
(out-of-stock parts already replaced there).

- Board outline extended 4.5 mm at the pin-1 end (35.7 -> 40.2 mm). The
  receptacle face sits flush with the new edge. The In2 +3V3 plane is
  stretched to match; the In1/In4 GND planes already covered it.
- New project footprint PicoROM:USB_C_Receptacle_HRO_TYPE-C-31-M-12, a
  copy of the KiCad 10 library footprint with the shield pads renamed
  SH -> S1 to match the schematic symbol (otherwise the shell would be
  left unconnected), the front silk line trimmed to the board edge, and
  the GCT USB4105 3D model as a stand-in (KiCad ships no HRO model).
- Old J1 escape routing removed and rerouted: both VBUS pad pairs to D4
  (linked on In3), CC1/CC2 to R6/R7, D+/D- pad pairs joined at the
  receptacle, GND pads to stitching vias. R7's GND via moved off the new
  A12/B1 pad. No other footprint moved.
- Title block revision 1.10 -> 1.10-S; back silkscreen date/version
  "Oct/26 v1.10-S". The front "v1.10" is unchanged: it already ends at
  U2's pads, so there is no room for a suffix.

DRC: 0 unconnected items and a clean schematic parity check; only the two
findings already present in 1.10 remain (U3/C3 courtyard overlap, U3
footprint type). The files in production/ are still the 1.10 outputs and
need regenerating before an order.

Co-Authored-By: Claude Opus 5.5 <noreply@anthropic.com>
Parts:
- J1: footprint Connector_USB:USB_C_Receptacle_G-Switch_GT-USB-7051x -> PicoROM:USB_C_Receptacle_HRO_TYPE-C-31-M-12; MPN C2843970 -> C165948
Changed lines of the file:
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@@
 	(title_block
 		(title "PicoROM-28 - ROM Emulator")
-		(date "2026-10-24")
-		(rev "1.10")
+		(date "2026-10-26")
+		(rev "1.10-S")
 		(company "Martin Donlon (@wickerwaka)")
 		(comment 1 "DIP-28 Form factor")
 		(comment 2 "Based on RP2040 minimal example")
+		(comment 3 "1.10-S: side-entry USB-C (HRO TYPE-C-31-M-12), board +4.5 mm at pin-1 end")
 	)
 	(text "Flash"
@@
 			)
 		)
-		(property "Footprint" "Connector_USB:USB_C_Receptacle_G-Switch_GT-USB-7051x"
+		(property "Footprint" "PicoROM:USB_C_Receptacle_HRO_TYPE-C-31-M-12"
 			(at 29.21 48.26 0)
 			(hide yes)
@@
 			)
 		)
-		(property "MPN" "C2843970"
+		(property "MPN" "C165948"
 			(at 25.4 48.26 0)
 			(hide yes)
