File: hardware/PicoROM-28/PicoROM-28.kicad_pcb (KiCad board)
At the start: 6 copper layers, 35.7 x 17.6 mm, 65 parts, among them J1 USB_C_Receptacle_USB2.0, J2 External Reset, J3 Conn_01x14, J4 Conn_01x14, J5 Conn_01x05_Pin, U1 NCP114AMX330TCG, U10 74LVC8245, U11 74AHCT1G126, U2 W25Q16JVUXIQ, U3 RP2040, U4 74LVC245, U5 74LVC245, U7 74AHCT1G126, U8 NCP114AMX330TCG, U9 74LVC245, Y1 ABM3-12.000MHZ-D2Y-T

Commit message: PicoROM-28 1.10-S: side-entry USB-C connector
Replace the vertical GT-USB-7051A USB-C receptacle (J1) with a horizontal
16-pin HRO TYPE-C-31-M-12 (LCSC C165948), so the plug enters from the
pin-1 end of the board instead of from above. Based on upstream 1.10
(out-of-stock parts already replaced there).

- Board outline extended 4.5 mm at the pin-1 end (35.7 -> 40.2 mm). The
  receptacle face sits flush with the new edge. The In2 +3V3 plane is
  stretched to match; the In1/In4 GND planes already covered it.
- New project footprint PicoROM:USB_C_Receptacle_HRO_TYPE-C-31-M-12, a
  copy of the KiCad 10 library footprint with the shield pads renamed
  SH -> S1 to match the schematic symbol (otherwise the shell would be
  left unconnected), the front silk line trimmed to the board edge, and
  the GCT USB4105 3D model as a stand-in (KiCad ships no HRO model).
- Old J1 escape routing removed and rerouted: both VBUS pad pairs to D4
  (linked on In3), CC1/CC2 to R6/R7, D+/D- pad pairs joined at the
  receptacle, GND pads to stitching vias. R7's GND via moved off the new
  A12/B1 pad. No other footprint moved.
- Title block revision 1.10 -> 1.10-S; back silkscreen date/version
  "Oct/26 v1.10-S". The front "v1.10" is unchanged: it already ends at
  U2's pads, so there is no room for a suffix.

DRC: 0 unconnected items and a clean schematic parity check; only the two
findings already present in 1.10 remain (U3/C3 courtyard overlap, U3
footprint type). The files in production/ are still the 1.10 outputs and
need regenerating before an order.

Co-Authored-By: Claude Opus 5.5 <noreply@anthropic.com>
Parts:
- J1: footprint Connector_USB:USB_C_Receptacle_G-Switch_GT-USB-7051x -> PicoROM:USB_C_Receptacle_HRO_TYPE-C-31-M-12
- moved J1 3.85 mm to (124.7, 64.7)
Routing:
- net Net-(D4-A): track 14.9 -> 10.7 mm
- net /USB_D+: track 22.2 -> 23.4 mm
- net Net-(J1-CC1): track 3.64 -> 4.33 mm
- net GND: track 62.8 -> 63.4 mm, vias 44 -> 41
- net /USB_D-: track 23.5 -> 23.7 mm, vias 3 -> 2
Other:
- board size 35.7 x 17.6 mm -> 40.2 x 17.6 mm
- board text added: "Oct/26 v1.10-S"
- board text removed: "Oct/2026 v1.10"

Commit message: PicoROM-28 1.10-S: remove branding from the silkscreen
Remove the PicoROM-28 text and the PicoROM logos from both sides, the QR
code, and the @wickerwaka handle from the back. Also remove the DIP-notch
circle, which the side-entry connector now covers.

Copper, mask, paste, outline and drill data are unchanged. The kicad-cli
JLCPCB outputs are regenerated: only the two silkscreen gerbers and the
designator list (logo footprints) change; BOM, CPL and IPC netlist are
identical.

Co-Authored-By: Claude Opus 5.5 <noreply@anthropic.com>
Parts:
- removed G***: LOGO, PicoROM:project_logo
- removed G***: LOGO, PicoROM:project_logo_large
- removed G***: LOGO, PicoROM:project_qrcode
Other:
- board text removed: "@wickerwaka"
- board text removed: "PicoROM-28"
